File: EMU-CAN-Splitter.kicad_sch (KiCad schematic)
At the start: 3 parts, among them J1 Conn_02x02_Top_Bottom, U1 XT30PW (2+2), U2 XT30PW (2+2)

Commit message: final
Parts:
- added H1, H2, H3, H4: MountingHole, MountingHole:MountingHole_3.2mm_M3_DIN965, symbol Mechanical:MountingHole
