File: EMU-CAN-Splitter.kicad_pcb (KiCad board)
At the start: 2 copper layers, 3 parts, among them J1 Conn_02x02_Top_Bottom, U1 XT30PW (2+2), U2 XT30PW (2+2)

Commit message: final
Parts:
- added H1: MountingHole, MountingHole:MountingHole_3.2mm_M3_DIN965, F.Cu at (99.5, 69.4)
- added H5: MountingHole, MountingHole:MountingHole_3.2mm_M3_DIN965, F.Cu at (127.5, 69.4)
- added H6: MountingHole, MountingHole:MountingHole_3.2mm_M3_DIN965, F.Cu at (99.5, 95.4)
- added H7: MountingHole, MountingHole:MountingHole_3.2mm_M3_DIN965, F.Cu at (127.5, 95.4)
Routing:
- net Net-(J1-Pin_1): track 26.7 -> 0.00 mm
- net Net-(J1-Pin_2): track 37.8 -> 39.6 mm
- added copper zone on F.Cu, net Net-(J1-Pin_1)
Other:
- board outline added: 36.7 x 36.1 mm

Commit message: Fix fill
Routing:
- added copper zone on B.Cu, net Net-(J1-Pin_1)
